File: getting_started/getting_started.kicad_sch (KiCad schematic)
At the start: 0 parts

Commit message: Updated KiCAD project
Parts:
- added BT1: Battery_Cell, Battery:BatteryHolder_Keystone_1058_1x2032, symbol Device:Battery_Cell
- added D1: LED, LED_THT:LED_D5.0mm, symbol Device:LED
- added R1: R_US, Resistor_THT:R_Axial_DIN0309_L9.0mm_D3.2mm_P12.70mm_Horizontal, symbol Device:R_US
Connections:
- new net GND: BT1.2 (-), D1.1 (K)
- new net VCC: BT1.1 (+), R1.1
- new net led: D1.2 (A), R1.2
Other:
- title: (none) -> Example Project
